File: weather_wifi.kicad_pcb (KiCad board)
At the start: 2 copper layers, 41.7 x 31.6 mm, 46 parts, among them J1 FPC 1x18, J2 USB2.0_type_c, Q1 S8050, Q2 S8050, Q3 AO3401A, SW1 key_reset/user, SW2 key_flash, U1 XC6206PxxxMR, U2 ESP8266EX, U3 W25Q32 4Mb flash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

Commit message: update for jlc manufacture
Parts:
- added REF**: MountingHole_1.152mm, weather_wifi:JLCPCB_MountingHole_1.152mm, F.Cu at (83.3, 66.4)
- renumbered G*** to G1
Other:
- board text added: "JLCJLCJLCJLC"
